File: Flute_hw/Flute.kicad_pcb (KiCad board)
At the start: 4 copper layers, 310.5 x 21.4 mm, 104 parts, among them Q1 IRLML6401, Q2 IRLML6401, SW1 BUTTON, SW2 BUTTON, SW3 BUTTON, SW4 BUTTON, SW5 BUTTON, SW6 BUTTON, SW7 BUTTON

Commit message: PCB sent to production
Parts:
- ANT1: footprint Antennas:Flute_868 -> Antennas:Flute_868_inverted
- C10, C11, C12, C13, C14, C15, C16, C17, C18, C19, C20, C21, C22, C23, C24, C25, C26, C27, C28, C29, C3, C30, C31, C32, C33, C34, C35, C36, C37, C38, C39, C4, C40, C41, C42, C43, C44, C45, C46, C47, C48, C5, C6, C7, C8, C9: footprint Capacitors:CAP_0603 -> Capacitors:CAP_0603_Silks
- L3: value BLM15 -> BLM15AG102SN1
- moved Logo1 19.2 mm to (349.1, 141.5)
- moved C1 7.76 mm to (328.0, 149.5), turned to -90 degrees
- moved C2 6.99 mm to (331.3, 148.5)
- moved L1 6.89 mm to (329.7, 149.0)
- moved C10 5.29 mm to (325.8, 151.1), turned to -90 degrees
- moved BLN1 4.80 mm to (326.1, 148.2)
- moved C13 4.80 mm to (315.9, 148.4)
- moved C5 4.80 mm to (318.9, 141.4)
- moved C6 4.80 mm to (324.9, 141.4)
- moved C7 4.80 mm to (315.9, 146.8)
- moved R3 4.80 mm to (317.1, 141.4)
- moved R5 4.80 mm to (321.9, 153.6)
- moved XTAL2 4.80 mm to (321.9, 141.4)
- moved C12 4.80 mm to (321.7, 144.0)
- moved C14 4.80 mm to (320.3, 153.6)
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Routing:
- net GND: track 0.00 -> 671.8 mm, vias 0 -> 298
- net +3v3: track 0.00 -> 253.5 mm, vias 0 -> 9
- net Net-(DD2-Pad26): track 0.00 -> 170.3 mm, vias 0 -> 1
- net /D-: track 0.00 -> 165.1 mm
- net /D+: track 0.00 -> 165.0 mm
- net /5V_USB: track 0.00 -> 136.6 mm, vias 0 -> 1
- net /SPK_M: track 0.00 -> 111.7 mm, vias 0 -> 5
- net /SPK_P: track 0.00 -> 110.8 mm, vias 0 -> 5
- net /BTN7: track 0.00 -> 103.2 mm, vias 0 -> 2
- net /CC_CS: track 0.00 -> 95.3 mm, vias 0 -> 2
- net /CC_MOSI: track 0.00 -> 93.5 mm, vias 0 -> 2
- net /CC_MISO: track 0.00 -> 92.9 mm, vias 0 -> 2
- net /CC_SCK: track 0.00 -> 91.9 mm, vias 0 -> 2
- net /CC_GDO0: track 0.00 -> 91.8 mm, vias 0 -> 2
- net /BTN6: track 0.00 -> 75.0 mm, vias 0 -> 2
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- added copper zone on B.Cu, net /SPK_M
- added copper zone on In1.Cu, net /SPK_M
- added copper zone on B.Cu, net /SPK_P
- added copper zone on In1.Cu, net /SPK_P
- added copper zone on B.Cu, net GND
- added copper zone on F.Cu, net GND
- added copper zone on In1.Cu, net GND
- added copper zone on In2.Cu, net GND
Other:
- board text added: "+"
- board text added: "GND"
- board text added: "Ostranna Flute 1.0"
- board text added: "SPK_M"
- board text added: "SPK_P"
