File: Flute_hw/Flute.kicad_sch (KiCad schematic)
At the start: 97 parts, among them Q1 IRLML6401, Q2 IRLML6401, SW1 BUTTON, SW2 BUTTON, SW3 BUTTON, SW4 BUTTON, SW5 BUTTON, SW6 BUTTON, SW7 BUTTON

Commit message: + Layout done
Parts:
- removed XL4: CONN_2, Connectors:SLD_2_2D5_1mm, symbol Connectors_kl:CONN_2
- removed XL5: CONN_2, Connectors:WB-02R(MW-2MR), symbol Connectors_kl:CONN_2
- added C48: 0.1u, Capacitors:CAP_0603, symbol Tittar_kl:C
- added HOLE5, HOLE6, HOLE7, HOLE8: HOLE_METALLED, PCB:Hole2d2_out3d5mm, symbol pcb_details:HOLE_METALLED
- added XL4, XL5: CONN_1, PCB:Oval3x1.5, symbol Connectors_kl:CONN_1
- added XL7, XL8: CONN_1, PCB:Square_1MM5, symbol Connectors_kl:CONN_1
- ANT1: footprint Radio:ANT_868_SEIDHE -> Antennas:Flute_868
- HOLE1, HOLE2, HOLE3, HOLE4: footprint PCB:Hole2d4_out4d5mm -> PCB:Hole2d2_out3d5mm
- XL1: footprint Connectors:PLS-6-NoHole -> Connectors:PLS-6_LOCK
- XL2: footprint Installation:MICROSD_EJECTOR_TFWF1 -> Installation:MICROSD_CAP_FIX05A
Connections:
- net +3v3: now also C48.2
- net +BATT: now also XL7.1 (P1)
- net GND: now also C48.1, HOLE5.H, HOLE6.H, HOLE7.H, HOLE8.H, XL8.1 (P1)
- net SPK_M: now also XL5.1 (P1)
- net SPK_P: now also XL4.1 (P1)
Other:
- moved on the sheet: HOLE1, HOLE2, HOLE3, HOLE4

Commit message: PCB sent to production
Parts:
- ANT1: footprint Antennas:Flute_868 -> Antennas:Flute_868_inverted
- C10, C11, C12, C13, C14, C15, C16, C17, C18, C19, C20, C21, C22, C23, C24, C25, C26, C27, C28, C29, C3, C30, C31, C32, C33, C34, C35, C36, C37, C38, C39, C4, C40, C41, C42, C43, C44, C45, C46, C47, C48, C5, C6, C7, C8, C9: footprint Capacitors:CAP_0603 -> Capacitors:CAP_0603_Silks
- L3: value BLM15 -> BLM15AG102SN1
